File: schemes/MotorController/MotorController.sch (KiCad schematic (older format))
At the start: 2 parts, among them U1 MD10-POT

Commit message: Added full schematics
Parts:
- added M1: Motor_DC, symbol Motor:Motor_DC
Connections:
- wire segments 8 -> 12
- no-connect marks 29 -> 27
Other:
- moved on the sheet: A1, U1
Changed lines of the file:
@@
 L MCU_Module:Arduino_UNO_R3 A1
 U 1 1 607028FB
-P 4150 3750
-F 0 "A1" H 5150 4650 50  0000 C CNN
-F 1 "Arduino_UNO_R3" H 5150 4550 50  0000 C CNN
-F 2 "Module:Arduino_UNO_R3" H 4150 3750 50  0001 C CIN
-F 3 "https://www.arduino.cc/en/Main/arduinoBoardUno" H 4150 3750 50  0001 C CNN
-	1    4150 3750
+P 5400 3600
+F 0 "A1" H 6400 4500 50  0000 C CNN
+F 1 "Arduino_UNO_R3" H 6400 4400 50  0000 C CNN
+F 2 "Module:Arduino_UNO_R3" H 5400 3600 50  0001 C CIN
+F 3 "https://www.arduino.cc/en/Main/arduinoBoardUno" H 5400 3600 50  0001 C CNN
+	1    5400 3600
 	-1   0    0    -1
 $EndComp
@@
 L MotorDriver:MD10-POT U1
 U 1 1 60706B4A
-P 5900 3100
-F 0 "U1" H 5925 3165 50  0000 C CNN
-F 1 "MD10-POT" H 5925 3074 50  0000 C CNN
-F 2 "" H 5400 3150 50  0001 C CNN
-F 3 "" H 5400 3150 50  0001 C CNN
-	1    5900 3100
+P 7850 2950
+F 0 "U1" H 7875 3015 50  0000 C CNN
+F 1 "MD10-POT" H 7875 2924 50  0000 C CNN
+F 2 "" H 7350 3000 50  0001 C CNN
+F 3 "" H 7350 3000 50  0001 C CNN
+	1    7850 2950
 	1    0    0    -1
 $EndComp
 Wire Wire Line
-	5000 3550 4650 3550
+	6100 3300 6100 3500
 Wire Wire Line
-	5000 3450 4850 3450
+	6100 3500 5900 3500
 Wire Wire Line
-	4850 3450 4850 3650
+	6000 3200 6000 4900
 Wire Wire Line
-	4850 3650 4650 3650
+	6000 4900 5500 4900
 Wire Wire Line
-	5000 3350 4750 3350
-Wire Wire Line
-	4750 3350 4750 5050
-Wire Wire Line
-	4750 5050 4250 5050
-Wire Wire Line
-	4250 5050 4250 4850
-NoConn ~ 3650 3150
-NoConn ~ 3650 3350
-NoConn ~ 3650 3550
-NoConn ~ 3650 3750
-NoConn ~ 3650 3850
-NoConn ~ 3650 3950
-NoConn ~ 3650 4050
-NoConn ~ 3650 4150
-NoConn ~ 3650 4250
-NoConn ~ 3650 4450
-NoConn ~ 4050 4850
-NoConn ~ 4150 4850
-NoConn ~ 3950 2750
-NoConn ~ 4050 2750
+	5500 4900 5500 4700
+NoConn ~ 4900 3000
+NoConn ~ 4900 3200
+NoConn ~ 4900 3400
+NoConn ~ 4900 3600
+NoConn ~ 4900 3700
+NoConn ~ 4900 3800
+NoConn ~ 4900 3900
+NoConn ~ 4900 4000
+NoConn ~ 4900 4100
+NoConn ~ 4900 4300
+NoConn ~ 5300 4700
+NoConn ~ 5400 4700
+NoConn ~ 5200 2600
 $Comp
 L power:+5V #PWR0101
 U 1 1 60719766
-P 4250 2750
-F 0 "#PWR0101" H 4250 2600 50  0001 C CNN
-F 1 "+5V" H 4265 2923 50  0000 C CNN
-F 2 "" H 4250 2750 50  0001 C CNN
-F 3 "" H 4250 2750 50  0001 C CNN
-	1    4250 2750
+P 5500 2600
+F 0 "#PWR0101" H 5500 2450 50  0001 C CNN
+F 1 "+5V" H 5515 2773 50  0000 C CNN
+F 2 "" H 5500 2600 50  0001 C CNN
+F 3 "" H 5500 2600 50  0001 C CNN
+	1    5500 2600
 	1    0    0    -1
 $EndComp
-NoConn ~ 6850 3400
-NoConn ~ 6850 3550
-NoConn ~ 3650 4550
-NoConn ~ 4650 4450
-NoConn ~ 4650 4350
-NoConn ~ 4650 4250
-NoConn ~ 4650 4150
-NoConn ~ 4650 4050
-NoConn ~ 4650 3950
-NoConn ~ 4650 3850
-NoConn ~ 4650 3750
-NoConn ~ 4650 3450
-NoConn ~ 4650 3350
-NoConn ~ 4650 3250
-NoConn ~ 4650 3150
+NoConn ~ 4900 4400
+NoConn ~ 5900 4300
+NoConn ~ 5900 4200
+NoConn ~ 5900 4100
+NoConn ~ 5900 4000
+NoConn ~ 5900 3800
+NoConn ~ 5900 3700
+NoConn ~ 5900 3600
+NoConn ~ 5900 3300
+NoConn ~ 5900 3200
+NoConn ~ 5900 3100
+NoConn ~ 5900 3000
 $Comp
-L power:-12V #PWR?
+L power:-12V #PWR0102
 U 1 1 6071C6B6
-P 6850 4000
-F 0 "#PWR?" H 6850 4100 50  0001 C CNN
-F 1 "-12V" V 6865 4128 50  0000 L CNN
-F 2 "" H 6850 4000 50  0001 C CNN
-F 3 "" H 6850 4000 50  0001 C CNN
-	1    6850 4000
+P 8800 3850
+F 0 "#PWR0102" H 8800 3950 50  0001 C CNN
+F 1 "-12V" V 8815 3978 50  0000 L CNN
+F 2 "" H 8800 3850 50  0001 C CNN
+F 3 "" H 8800 3850 50  0001 C CNN
+	1    8800 3850
 	0    1    1    0
 $EndComp
 $Comp
-L power:+12V #PWR?
+L power:+12V #PWR0103
 U 1 1 6071CF39
-P 6850 4150
-F 0 "#PWR?" H 6850 4000 50  0001 C CNN
-F 1 "+12V" V 6865 4278 50  0000 L CNN
-F 2 "" H 6850 4150 50  0001 C CNN
-F 3 "" H 6850 4150 50  0001 C CNN
-	1    6850 4150
+P 8800 4000
+F 0 "#PWR0103" H 8800 3850 50  0001 C CNN
+F 1 "+12V" V 8815 4128 50  0000 L CNN
+F 2 "" H 8800 4000 50  0001 C CNN
+F 3 "" H 8800 4000 50  0001 C CNN
+	1    8800 4000
 	0    1    1    0
 $EndComp
+Wire Wire Line
+	6000 3200 6950 3200
+Wire Wire Line
+	6100 3300 6950 3300
+Wire Wire Line
+	5900 3400 6950 3400
+$Comp
+L Motor:Motor_DC M1
+U 1 1 609FEB04
+P 9200 3250
+F 0 "M1" H 9358 3246 50  0000 L CNN
+F 1 "Motor_DC" H 9358 3155 50  0000 L CNN
+F 2 "" H 9200 3160 50  0001 C CNN
+F 3 "~" H 9200 3160 50  0001 C CNN
+	1    9200 3250
+	1    0    0    -1
+$EndComp
+Wire Wire Line
+	8800 3250 8800 3050
+Wire Wire Line
+	8800 3050 9200 3050
+Wire Wire Line
+	8800 3400 8800 3550
+Wire Wire Line
+	8800 3550 9200 3550
+NoConn ~ 5300 2600
+NoConn ~ 5900 3900
 $EndSCHEMATC
